File: _autosave-OpenC64Cart.kicad_pcb (KiCad board)
At the start: 2 copper layers, 58.4 x 50.8 mm, 17 parts, among them J99 PEG_HOLE, SW1 RESET_SW, SW101 SW_Coded_SH-7010, U1 C64-Exp-Port, U101 74LS02, U102 4066, U2 27512

Commit message: OpenC64DiagCart
Initial commit of OpenC64DiagCart fork.
Other:
- board text added: "Slot 0 Dead Test 781220 1 C64 Diag. 586220* 2 Roßmöller Doctor64 3 Trilogic 64 Doctor"
- board text added: "Slot 4 C64 Burn In 5 1541 Diagnostic 6 PSID64 Sid Player 7 586220* (SWINSID)"
- board text removed: "Slot 0 TEST1 1 TEST1 2 TEST1 3 TEST1"
- board text removed: "Slot 4 TEST1 5 TEST1 6 TEST1 7 TEST1"
Changed lines of the file:
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@@
       (net 1 GND))
   )
-  (gr_line (start 93.218 102.87) (end 93.218 111.506) (layer B.SilkS) (width 0.15))
-  (gr_line (start 110.998 102.87) (end 110.998 111.506) (layer B.SilkS) (width 0.15))
-  (gr_text "Slot\n 4   TEST1\n 5   TEST1\n 6   TEST1\n 7   TEST1" (at 96.52 107.188) (layer B.SilkS)
+  (gr_line (start 92.964 102.87) (end 92.964 111.506) (layer B.SilkS) (width 0.15))
+  (gr_line (start 112.522 102.87) (end 112.522 111.506) (layer B.SilkS) (width 0.15))
+  (gr_text " Slot\n  4   C64 Burn In\n  5   1541 Diagnostic\n  6   PSID64 Sid Player\n  7   586220* (SWINSID)" (at 97.028 107.188) (layer B.SilkS)
     (effects (font (size 1 1) (thickness 0.15)) (justify left mirror))
   )
-  (gr_line (start 96.52 102.87) (end 96.52 111.506) (layer B.SilkS) (width 0.15))
-  (gr_line (start 114.3 104.648) (end 80.01 104.648) (layer B.SilkS) (width 0.15))
-  (gr_text "Slot\n 0   TEST1\n 1   TEST1\n 2   TEST1\n 3   TEST1" (at 114.3 107.188) (layer B.SilkS)
+  (gr_line (start 96.266 102.87) (end 96.266 111.506) (layer B.SilkS) (width 0.15))
+  (gr_line (start 115.824 104.648) (end 77.47 104.648) (layer B.SilkS) (width 0.15))
+  (gr_text "Slot\n 0   Dead Test 781220\n 1   C64 Diag. 586220*\n 2   Roßmöller Doctor64\n 3   Trilogic 64 Doctor" (at 115.824 107.188) (layer B.SilkS)
     (effects (font (size 1 1) (thickness 0.15)) (justify left mirror))
   )
-  (gr_line (start 80.01 111.506) (end 80.01 102.87) (layer B.SilkS) (width 0.15))
-  (gr_line (start 114.3 111.506) (end 80.01 111.506) (layer B.SilkS) (width 0.15))
-  (gr_line (start 114.3 102.87) (end 114.3 111.506) (layer B.SilkS) (width 0.15))
-  (gr_line (start 80.01 102.87) (end 114.3 102.87) (layer B.SilkS) (width 0.15))
+  (gr_line (start 77.47 111.506) (end 77.47 102.87) (layer B.SilkS) (width 0.15))
+  (gr_line (start 115.824 111.506) (end 77.47 111.506) (layer B.SilkS) (width 0.15))
+  (gr_line (start 115.824 102.87) (end 115.824 111.506) (layer B.SilkS) (width 0.15))
+  (gr_line (start 77.47 102.87) (end 115.824 102.87) (layer B.SilkS) (width 0.15))
   (dimension 8.809086 (width 0.15) (layer Cmts.User)
     (gr_text "8.809 mm" (at 113.776865 84.85103 2.602562202) (layer Cmts.User)
