File: OpenC64Cart.sch (KiCad schematic (older format))
At the start: 17 parts, among them J99 PEG_HOLE, SW1 RESET_SW, SW101 SW_Coded_SH-7010, U1 C64-Exp-Port, U101 74LS02, U102 4066, U2 27512

Commit message: Fixed Everything
This is still untested beta. I had a bunch of things wrong on my first test PCBs.
Connections:
- net +5V: now also U102.14 (VDD); no longer U102.7 (VSS)
- net GND: now also U102.7 (VSS); no longer U102.14 (VDD)
- net ROMH: now reaches U102.1
- net ROMH: now also U1.B (/ROMH); no longer U1.11 (/ROML)
- net EXROM: now reaches U101.11, U101.12, U101.4, U102.12, U102.13
- net EXROM: now also U1.9 (/EXROM); no longer U1.8 (/GAME)
- net GAME: now reaches U101.13, U102.5, U102.6
- net GAME: now also U1.8 (/GAME); no longer U1.9 (/EXROM)
- net ROML: now reaches U102.4
- net ROML: now also U1.11 (/ROML); no longer U1.B (/ROMH)
- net CE: now reaches U102.2, U2.20 (CE), U2.22 (OE)
- net CE: now also U102.3
- net at U101.1: now also U101.8, U101.9
Other:
- moved on the sheet: U102B
Changed lines of the file:
@@
 $EndDescr
-$Comp
-L C64-Exp-Port:C64-Exp-Port U1
-U 1 1 59713F4B
-P 4381 3340
-F 0 "U1" H 4381 3240 50  0000 C CNN
-F 1 "C64-Exp-Port" H 4381 4640 50  0000 C CNN
-F 2 "OpenC64Cart:C64-Cart" H 4381 3340 50  0001 C CNN
-F 3 "https://www.c64-wiki.com/wiki/Expansion_Port" H 4381 3340 50  0001 C CNN
-	1    4381 3340
-	-1   0    0    1
-$EndComp
 $Comp
 L Device:C C1
@@
 Wire Wire Line
 	8381 4040 8381 4140
-Wire Wire Line
-	8381 4140 8531 4140
-Connection ~ 8381 4140
-Wire Wire Line
-	3631 4290 3331 4290
-Wire Wire Line
-	5131 3390 6131 3390
-Wire Wire Line
-	6131 3390 6131 5287
 NoConn ~ 5131 3190
 NoConn ~ 5131 3290
@@
 	5331 1940 5631 1940
 Wire Wire Line
-	8381 4140 8381 5740
-Wire Wire Line
 	2981 4190 3631 4190
 Wire Wire Line
@@
 	1    1636 4837
 	1    0    0    -1
-$EndComp
-$Comp
-L 4xxx:4066 U102
-U 1 1 6195B65C
-P 2554 5753
-F 0 "U102" H 2554 5580 50  0000 C CNN
-F 1 "4066" H 2554 5489 50  0000 C CNN
-F 2 "Package_DIP:DIP-14_W7.62mm" H 2554 5753 50  0001 C CNN
-F 3 "http://www.ti.com/lit/ds/symlink/cd4066b.pdf" H 2554 5753 50  0001 C CNN
-	1    2554 5753
-	0    -1   1    0
-$EndComp
-$Comp
-L 4xxx:4066 U102
-U 2 1 6195CC77
-P 2554 6352
-F 0 "U102" H 2554 6179 50  0000 C CNN
-F 1 "4066" H 2554 6088 50  0000 C CNN
-F 2 "Package_DIP:DIP-14_W7.62mm" H 2554 6352 50  0001 C CNN
-F 3 "http://www.ti.com/lit/ds/symlink/cd4066b.pdf" H 2554 6352 50  0001 C CNN
-	2    2554 6352
-	0    -1   -1   0
 $EndComp
 $Comp
@@
 A15
 Wire Wire Line
-	1937 4837 2149 4837
-Wire Wire Line
 	2149 4837 2149 6688
 Wire Wire Line
@@
 Wire Wire Line
 	2083 6162 2083 5753
-Wire Wire Line
-	1929 6351 2254 6351
-Wire Wire Line
-	2254 6351 2254 6352
-Wire Wire Line
-	2083 5753 2254 5753
 Connection ~ 2083 5753
 Wire Wire Line
 	2083 5753 2083 5373
-Wire Wire Line
-	2554 6053 4008 6053
-Wire Wire Line
-	4008 6053 4008 5740
-Wire Wire Line
-	4008 5740 8381 5740
 Wire Wire Line
 	1928 5373 2083 5373
 Connection ~ 2083 5373
 Wire Wire Line
-	2083 5373 2253 5373
-Wire Wire Line
-	5924 5494 3050 5494
-Wire Wire Line
-	3050 5494 3050 6869
-Wire Wire Line
 	3050 6869 2255 6869
 Wire Wire Line
 	1929 6351 1928 6351
-Wire Wire Line
-	1929 6351 1929 6869
-Connection ~ 1929 6351
-Wire Wire Line
-	5129 3590 5131 3590
-$Comp
-L 4xxx:4066 U102
-U 5 1 61C253FE
-P 4319 6953
-F 0 "U102" V 3952 6953 50  0000 C CNN
-F 1 "4066" V 4043 6953 50  0000 C CNN
-F 2 "Package_DIP:DIP-14_W7.62mm" H 4319 6953 50  0001 C CNN
-F 3 "http://www.ti.com/lit/ds/symlink/cd4066b.pdf" H 4319 6953 50  0001 C CNN
-	5    4319 6953
-	0    1    1    0
-$EndComp
 $Comp
 L power:GND #PWR0107
@@
 	0    1    1    0
 $EndComp
-Wire Wire Line
-	5924 3590 5131 3590
-Wire Wire Line
-	5924 3590 5924 5494
-Connection ~ 5131 3590
-Wire Wire Line
-	5131 3690 6011 3690
-Wire Wire Line
-	6011 3690 6011 5373
-Wire Wire Line
-	2554 5453 2554 5287
-Wire Wire Line
-	2554 5287 6131 5287
-Wire Wire Line
-	3331 4290 3331 6652
-Wire Wire Line
-	3331 6652 2554 6652
 $Comp
 L 4xxx:4066 U102
@@
 Wire Wire Line
 	2253 4915 2253 5373
-Connection ~ 2253 5373
-Wire Wire Line
-	2253 5373 6011 5373
 $Comp
 L Device:LED D2
@@
 $EndComp
 NoConn ~ 9461 6042
+Wire Wire Line
+	2083 5753 2254 5753
+$Comp
+L 4xxx:4066 U102
+U 1 1 6195B65C
+P 2554 5753
+F 0 "U102" H 2554 5580 50  0000 C CNN
+F 1 "4066" H 2554 5489 50  0000 C CNN
+F 2 "Package_DIP:DIP-14_W7.62mm" H 2554 5753 50  0001 C CNN
+F 3 "http://www.ti.com/lit/ds/symlink/cd4066b.pdf" H 2554 5753 50  0001 C CNN
+	1    2554 5753
+	0    -1   1    0
+$EndComp
+$Comp
+L 4xxx:4066 U102
+U 5 1 61C253FE
+P 4319 6953
+F 0 "U102" V 3952 6953 50  0000 C CNN
+F 1 "4066" V 4043 6953 50  0000 C CNN
+F 2 "Package_DIP:DIP-14_W7.62mm" H 4319 6953 50  0001 C CNN
+F 3 "http://www.ti.com/lit/ds/symlink/cd4066b.pdf" H 4319 6953 50  0001 C CNN
+	5    4319 6953
+	0    -1   -1   0
+$EndComp
+Wire Wire Line
+	2554 6072 2554 6065
+$Comp
+L 4xxx:4066 U102
+U 2 1 6195CC77
+P 2554 6372
+F 0 "U102" H 2554 6199 50  0000 C CNN
+F 1 "4066" H 2554 6108 50  0000 C CNN
+F 2 "Package_DIP:DIP-14_W7.62mm" H 2554 6372 50  0001 C CNN
+F 3 "http://www.ti.com/lit/ds/symlink/cd4066b.pdf" H 2554 6372 50  0001 C CNN
+	2    2554 6372
+	0    -1   -1   0
+$EndComp
+Text Label 3631 4290 2    60   ~ 0
+ROMH
+Text Label 5131 3390 0    60   ~ 0
+ROML
+Text Label 5131 3590 0    60   ~ 0
+EXROM
+$Comp
+L C64-Exp-Port:C64-Exp-Port U1
+U 1 1 59713F4B
+P 4381 3340
+F 0 "U1" H 4381 3240 50  0000 C CNN
+F 1 "C64-Exp-Port" H 4381 4640 50  0000 C CNN
+F 2 "OpenC64Cart:C64-Cart" H 4381 3340 50  0001 C CNN
+F 3 "https://www.c64-wiki.com/wiki/Expansion_Port" H 4381 3340 50  0001 C CNN
+	1    4381 3340
+	-1   0    0    1
+$EndComp
+Text Label 5131 3690 0    60   ~ 0
+GAME
+Wire Wire Line
+	2083 5373 2253 5373
+Connection ~ 2253 5373
+Wire Wire Line
+	2253 5373 3058 5373
+Wire Wire Line
+	1929 4837 1936 4837
+Connection ~ 1936 4837
+Wire Wire Line
+	1936 4837 2149 4837
+Text Label 2554 6672 0    60   ~ 0
+ROML
+Text Label 2554 5453 0    60   ~ 0
+ROMH
+Text Label 3050 6869 0    60   ~ 0
+GAME
+Text Label 3058 5373 0    60   ~ 0
+EXROM
+Wire Wire Line
+	1929 6351 1929 6869
+Wire Wire Line
+	1928 6372 1928 6351
+Wire Wire Line
+	1928 6372 2254 6372
+Connection ~ 1928 6351
+Wire Wire Line
+	2554 6065 2605 6065
+Connection ~ 2554 6065
+Wire Wire Line
+	2554 6065 2554 6053
+Text Label 2605 6065 0    60   ~ 0
+CE
+Text Label 8297 4140 2    60   ~ 0
+CE
+Wire Wire Line
+	8297 4140 8381 4140
+Connection ~ 8381 4140
+Wire Wire Line
+	8381 4140 8531 4140
 $EndSCHEMATC
